File: motion-sensor-hardware.kicad_pcb (KiCad board)
At the start: 2 copper layers, 76.2 x 50.8 mm, 10 parts, among them Q1 BSS138, U1 ESP32-DevKitC, U2 LD2410C

Commit message: Added car charger circuits
Parts:
- removed Q1: BSS138, Package_TO_SOT_SMD:SOT-23
- added C10: 0.1u, Capacitor_SMD:C_0805_2012Metric, F.Cu at (340.9, 108.6)
- added C11: 0.1u, Capacitor_SMD:C_0805_2012Metric, F.Cu at (340.9, 111.6)
- added C2: 0.1u, Capacitor_SMD:C_0805_2012Metric, F.Cu at (336.5, 108.6)
- added C3: 22u, Capacitor_SMD:C_0805_2012Metric, F.Cu at (336.5, 111.6)
- added C4: 0.01u, Capacitor_SMD:C_0805_2012Metric, F.Cu at (336.5, 114.6)
- added C5: 1u, Capacitor_SMD:C_0805_2012Metric, F.Cu at (336.5, 117.7)
- added C6: 10u, Capacitor_SMD:C_0805_2012Metric, F.Cu at (336.5, 120.7)
- added C7: 1u, Capacitor_SMD:C_0805_2012Metric, F.Cu at (380.7, 59.4)
- added C8: 0.1u, Capacitor_SMD:C_0805_2012Metric, F.Cu at (380.7, 62.4)
- added C9: 22u, Capacitor_SMD:C_0805_2012Metric, F.Cu at (336.5, 123.7)
- added D2: LESD5D5.0CT1G, Diode_SMD:D_SOD-523, F.Cu at (370.8, 101.4)
- added D3: LESD5D5.0CT1G, Diode_SMD:D_SOD-523, F.Cu at (370.8, 103.9)
- added D5: PTVS20VS1UR,115, Diode_SMD:Nexperia_DSN1608-2_1.6x0.8mm, F.Cu at (378.7, 98.9)
- added J2: MX300-5.0-02P-BU01-Cu-Y-A, My_Connectors:MX300-5.0-02P, F.Cu at (340.0, 99.3)
- added J3: Conn_01x03, Connector_PinHeader_2.54mm:PinHeader_1x03_P2.54mm_Vertical, F.Cu at (383.0, 90.1)
- added J4: Conn_01x02, Connector_PinHeader_2.54mm:PinHeader_1x02_P2.54mm_Vertical, F.Cu at (374.9, 100.1)
- added J5: TYPE-C 16PIN 2MD(073), Connector_USB:USB_C_Receptacle_GCT_USB4105-xx-A_16P_TopMnt_Horizontal, F.Cu at (78.8, 94.5)
- added JP1: SolderJumper_3_Open, Jumper:SolderJumper-3_P1.3mm_Open_Pad1.0x1.5mm, F.Cu at (346.0, 120.2)
- added L1: 4.7uH, Inductors:IND_54x52, F.Cu at (346.9, 110.5)
- added R10: 0, Capacitor_SMD:C_0805_2012Metric, F.Cu at (89.0, 96.4)
- added R11: 10k, Capacitor_SMD:C_0805_2012Metric, F.Cu at (385.2, 68.4)
- added R2: 102k, Capacitor_SMD:C_0805_2012Metric, F.Cu at (340.9, 114.6)
- added R3: 18.7k, Capacitor_SMD:C_0805_2012Metric, F.Cu at (340.9, 117.7)
- added R4: 40.2k, Capacitor_SMD:C_0805_2012Metric, F.Cu at (340.9, 120.7)
- added R5: 5.1k, Capacitor_SMD:C_0805_2012Metric, F.Cu at (380.7, 68.4)
- added R6: 10k, Capacitor_SMD:C_0805_2012Metric, F.Cu at (380.7, 71.4)
- added R7: 10k, Capacitor_SMD:C_0805_2012Metric, F.Cu at (385.2, 56.4)
- added R8: 10k, Capacitor_SMD:C_0805_2012Metric, F.Cu at (385.2, 59.4)
- added R9: 0, Capacitor_SMD:C_0805_2012Metric, F.Cu at (89.0, 93.8)
- added SW1: SW_Push, Button_Switch_SMD:SW_Push_1P1T_NO_CK_KMR2, F.Cu at (381.8, 75.3)
- added SW2: SW_Push, Button_Switch_SMD:SW_Push_1P1T_NO_CK_KMR2, F.Cu at (381.8, 79.9)
- added U3: LT8608EMSE, Package_SO:MSOP-10-1EP_3x3mm_P0.5mm_EP1.68x1.88mm, F.Cu at (346.8, 116.2)
- added U4: TLV73333PDBV, Package_TO_SOT_SMD:SOT-23-5, F.Cu at (351.4, 120.8)
- C1: footprint Capacitor_SMD:C_0805_2012Metric_Pad1.18x1.45mm_HandSolder -> Capacitor_SMD:C_0805_2012Metric
- D1: value WS2812B -> LESD5D5.0CT1G; footprint LED_SMD:LED_WS2812B_PLCC4_5.0x5.0mm_P3.2mm -> Diode_SMD:D_SOD-523
- R1: value 10k -> 5.1k; footprint Resistor_SMD:R_0805_2012Metric_Pad1.20x1.40mm_HandSolder -> Capacitor_SMD:C_0805_2012Metric
- U1: value ESP32-DevKitC -> ESP32-C3-MINI-1-N4; footprint ESP32-DevkitC-32:ESP32-DevKitC -> RF_Module:ESP32-C6-MINI-1
- moved R1 266.6 mm to (380.7, 65.4), turned to 0 degrees
- moved C1 264.6 mm to (380.7, 56.4)
- moved D1 248.1 mm to (370.8, 99.0)
- moved U2 232.1 mm to (352.4, 89.8), turned to 0 degrees
- moved U1 9.14 mm to (94.6, 83.7)
Connections:
- C1 pad 1: +5V -> VUSB
- D1 pad 1: +5V -> GND
- D1 pad 2: unconnected-(D1-DOUT-Pad2) -> /USB1-
- R1 pad 1: +5V -> Net-(J5-CC1)
- R1 pad 2: Net-(D1-DIN) -> GND
- U1 pad 1: +3.3V -> GND
- U1 pad 11: unconnected-(U1-ADC2_CH7/GPIO27-Pad11) -> GND
- U1 pad 19: +5V -> /OUT
- U1 pad 2: unconnected-(U1-CHIP_PU-Pad2) -> GND
- U1 pad 20: unconnected-(U1-SD_CLK/GPIO6-Pad20) -> /RDR_RX
- U1 pad 21: unconnected-(U1-SD_DATA0/GPIO7-Pad21) -> /RDR_TX
- U1 pad 22: unconnected-(U1-SD_DATA1/GPIO8-Pad22) -> Net-(U1-GPIO8)
- U1 pad 23: unconnected-(U1-MTDO/GPIO15/ADC2_CH3-Pad23) -> Net-(U1-GPIO9)
- U1 pad 26: unconnected-(U1-ADC2_CH0/GPIO4-Pad26) -> /USB-
- U1 pad 27: unconnected-(U1-GPIO16-Pad27) -> /USB+
- U1 pad 3: unconnected-(U1-SENSOR_VP/GPIO36/ADC1_CH0-Pad3) -> +3.3V
- U1 pad 30: /RDR_RX -> Net-(J4-Pin_2)
- U1 pad 31: /RDR_TX -> Net-(J4-Pin_1)
- U1 pad 32: GND -> unconnected-(U1-NC-Pad32)
- U1 pad 33: /OUT -> unconnected-(U1-NC-Pad33)
- U1 pad 36: Net-(Q1-S) -> GND
- U1 pad 37: unconnected-(U1-GPIO23-Pad37) -> GND
- U1 pad 5: unconnected-(U1-VDET_1/GPIO34/ADC1_CH6-Pad5) -> Net-(U1-GPIO2/ADC1_CH2)
- U1 pad 8: unconnected-(U1-32K_XN/GPIO33/ADC1_CH5-Pad8) -> Net-(U1-EN/CHIP_PU)
Routing:
- net +5V: track 87.7 -> 0.00 mm
- net +3.3V: track 57.5 -> 0.00 mm, vias 1 -> 0
- net Net-(Q1-S): track 37.4 -> 0.00 mm, vias 1 -> 0
- net /USB+: track 0.00 -> 24.9 mm
- net /USB-: track 0.00 -> 23.6 mm
- net /OUT: track 19.0 -> 0.00 mm
- net /RDR_TX: track 17.6 -> 0.00 mm
- net Net-(D1-DIN): track 17.1 -> 0.00 mm
- net /RDR_RX: track 9.77 -> 0.00 mm
- net /USB1+: track 0.00 -> 3.59 mm
- net GND: track 3.39 -> 0.00 mm, vias 2 -> 0
- removed copper zone on B.Cu, net GND

Commit message: Split the two ground planes
Parts:
- removed the J2 at (340.0, 99.3)
- removed JP1: SolderJumper_3_Open, Jumper:SolderJumper-3_P1.3mm_Open_Pad1.0x1.5mm
- removed the U4 at (351.4, 120.8)
- added C12: 100nF, Capacitor_SMD:C_0603_1608Metric, F.Cu at (103.6, 107.0)
- added C13: 100nF, Capacitor_SMD:C_0603_1608Metric, F.Cu at (119.5, 107.0)
- added C14: 47uF, Capacitor_SMD:C_1206_3216Metric, F.Cu at (109.3, 101.5)
- added C15: 47uF, Capacitor_SMD:C_1206_3216Metric, F.Cu at (125.3, 106.8)
- added C16: 47uF, Capacitor_SMD:C_1206_3216Metric, F.Cu at (109.3, 106.8)
- added C17: 47uF, Capacitor_SMD:C_1206_3216Metric, F.Cu at (125.3, 101.5)
- added C19: 10uF, Capacitor_SMD:C_0603_1608Metric, F.Cu at (110.6, 81.1)
- added D4: WS2812B-HS01/W, LED_SMD:LED_WS2812B_PLCC4_5.0x5.0mm_P3.2mm, F.Cu at (116.3, 84.3)
- added F1: JK-nSMD100/16V, Fuse:Fuse_1206_3216Metric, F.Cu at (86.4, 111.5)
- added J1: MX128-2.54-02P, !Connectors:MX128-2.54-02P, F.Cu at (78.8, 111.5)
- added L2: FXL0630-6R8-M, Inductor_SMD:L_Changjiang_FXL0630, F.Cu at (119.5, 102.6)
- added Q1: AO3401A, Package_TO_SOT_SMD:TSOT-23, F.Cu at (91.5, 111.6)
- added R12: 20kΩ, Resistor_SMD:R_0603_1608Metric, F.Cu at (106.8, 107.8)
- added R13: 3.6kΩ, Resistor_SMD:R_0603_1608Metric, F.Cu at (106.8, 111.0)
- added R14: 49.9kΩ, Resistor_SMD:R_0603_1608Metric, F.Cu at (122.7, 107.8)
- added R15: 15kΩ, Resistor_SMD:R_0603_1608Metric, F.Cu at (122.7, 111.0)
- added U1: USBLC6-2SC6, Package_TO_SOT_SMD:SOT-23-6, F.Cu at (88.3, 94.5)
- added U5: SN74LV1T125DCK, Package_TO_SOT_SMD:SOT-353_SC-70-5, F.Cu at (107.4, 83.7)
- added U6: AP62200TWU-7, Package_TO_SOT_SMD:SOT-23-6, F.Cu at (103.6, 109.6)
- added U7: AP62200TWU-7, Package_TO_SOT_SMD:SOT-23-6, F.Cu at (119.5, 109.6)
- C1: value 0.1u -> 1uF; footprint Capacitor_SMD:C_0805_2012Metric -> Capacitor_SMD:C_0603_1608Metric
- C10, C11, C2, C8: value 0.1u -> 100nF; footprint Capacitor_SMD:C_0805_2012Metric -> Capacitor_SMD:C_0603_1608Metric
- C3, C9: value 22u -> 100nF; footprint Capacitor_SMD:C_0805_2012Metric -> Capacitor_SMD:C_0603_1608Metric
- C4: value 0.01u -> 10uF; footprint Capacitor_SMD:C_0805_2012Metric -> Capacitor_SMD:C_0603_1608Metric
- C5: value 1u -> 100nF; footprint Capacitor_SMD:C_0805_2012Metric -> Capacitor_SMD:C_0603_1608Metric
- C6: value 10u -> 10uF
- C7: value 1u -> 10uF
- D1: value LESD5D5.0CT1G -> P6SMB24CA-E3/52; footprint Diode_SMD:D_SOD-523 -> Diode_SMD:D_SMB
- D2: value LESD5D5.0CT1G -> BZT52C10S; footprint Diode_SMD:D_SOD-523 -> Diode_SMD:D_SOD-323
- D3: value LESD5D5.0CT1G -> SMF6.5CA; footprint Diode_SMD:D_SOD-523 -> Diode_SMD:D_SOD-123F
- D5: value PTVS20VS1UR,115 -> SMF6.5CA; footprint Diode_SMD:Nexperia_DSN1608-2_1.6x0.8mm -> Diode_SMD:D_SOD-123F
- J3: value Conn_01x03 -> PZ254V-11-03P
- J4: value Conn_01x02 -> MX128-2.54-04P; footprint Connector_PinHeader_2.54mm:PinHeader_1x02_P2.54mm_Vertical -> !Connectors:MX128-2.54-04P
- L1: value 4.7uH -> FXL0630-6R8-M; footprint Inductors:IND_54x52 -> Inductor_SMD:L_Changjiang_FXL0630
- R1: value 5.1k -> 5.1kΩ; footprint Capacitor_SMD:C_0805_2012Metric -> Resistor_SMD:R_0603_1608Metric
- R10, R9: value 0 -> 10kΩ; footprint Capacitor_SMD:C_0805_2012Metric -> Resistor_SMD:R_0603_1608Metric
- R11, R8: value 10k -> 10kΩ; footprint Capacitor_SMD:C_0805_2012Metric -> Resistor_SMD:R_0603_1608Metric
- R2: value 102k -> 5.1kΩ; footprint Capacitor_SMD:C_0805_2012Metric -> Resistor_SMD:R_0603_1608Metric
- R3: value 18.7k -> 100Ω; footprint Capacitor_SMD:C_0805_2012Metric -> Resistor_SMD:R_0603_1608Metric
- R4: value 40.2k -> 10kΩ; footprint Capacitor_SMD:C_0805_2012Metric -> Resistor_SMD:R_0603_1608Metric
- R5: value 5.1k -> 0Ω; footprint Capacitor_SMD:C_0805_2012Metric -> Resistor_SMD:R_0603_1608Metric
- R6: value 10k -> 0Ω; footprint Capacitor_SMD:C_0805_2012Metric -> Resistor_SMD:R_0603_1608Metric
- R7: value 10k -> 330Ω; footprint Capacitor_SMD:C_0805_2012Metric -> Resistor_SMD:R_0603_1608Metric
- SW1, SW2: value SW_Push -> TS-1088-AR02016; footprint Button_Switch_SMD:SW_Push_1P1T_NO_CK_KMR2 -> Button_Switch_SMD:SW_Push_SPST_NO_Alps_SKRK
- U2: value LD2410C -> ASSR-1218; footprint HLK:LD2410C -> Package_SO:SO-4_4.4x4.3mm_P2.54mm
- U3: value LT8608EMSE -> LD2410C; footprint Package_SO:MSOP-10-1EP_3x3mm_P0.5mm_EP1.68x1.88mm -> !Sensors:LD2410C
- U4: renamed from U1; footprint RF_Module:ESP32-C6-MINI-1 -> !RF_Modules:ESP32-C6-MINI-1
- moved R11 299.7 mm to (85.8, 83.0)
- moved R1 295.7 mm to (86.2, 91.2)
- moved D5 291.7 mm to (87.7, 118.0)
- moved R5 289.5 mm to (92.3, 93.5)
- moved R6 289.4 mm to (92.3, 95.5)
- moved C8 285.1 mm to (99.5, 109.6), turned to 90 degrees
- moved D1 284.5 mm to (86.4, 105.9), turned to -90 degrees
- moved R7 282.4 mm to (110.6, 122.4), turned to -90 degrees
- moved J4 280.7 mm to (95.1, 122.4), turned to 180 degrees
- moved R8 276.0 mm to (111.2, 93.2)
- moved D2 275.6 mm to (95.3, 107.8), turned to 90 degrees
- moved D3 272.3 mm to (99.1, 122.4), turned to -90 degrees
- moved C1 272.3 mm to (111.2, 95.1), turned to 180 degrees
- moved C7 271.7 mm to (113.7, 109.6), turned to 90 degrees
- moved SW1 266.6 mm to (115.8, 93.8), turned to 180 degrees
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- renumbered J5 to J2
Connections:
- C1 pad 1: VUSB -> Net-(U4-EN/CHIP_PU)
- C10 pad 1: +5V -> Net-(U6-EN)
- C11 pad 1: +3.3V -> Net-(U7-EN)
- C2 pad 1: Net-(U3-BST) -> +5V
- C2 pad 2: Net-(U3-SW) -> GND
- C3 pad 1: +5V -> +3.3V
- C4 pad 1: Net-(U3-TR/SS) -> +3.3V
- C5 pad 1: Net-(JP1-B) -> +5V
- C6 pad 1: /Voltage Regulator/VIN -> VIN
- C7 pad 1: Net-(U1-EN/CHIP_PU) -> VIN
- C8 pad 1: +3.3V -> VIN
- C9 pad 1: +3.3V -> VIN
- D1 pad 2: /USB1- -> Net-(D1-A2)
- D2 pad 1: GND -> VIN
- D2 pad 2: /USB1+ -> Net-(D2-A)
- D3 pad 1: GND -> /CTL_SW2
- D3 pad 2: VUSB -> /CTL_SW1
- D5 pad 1: VIN -> GND
- D5 pad 2: GND -> /STAT_SW
- J2 pad A4: VUSB -> Net-(U1-VBUS)
- J2 pad A6: /USB1+ -> Net-(J2-D+-PadA6)
- J2 pad A7: /USB1- -> Net-(J2-D--PadA7)
- J2 pad A9: VUSB -> Net-(U1-VBUS)
- J2 pad B4: VUSB -> Net-(U1-VBUS)
- J2 pad B5: Net-(J5-CC2) -> Net-(J2-CC2)
- J2 pad B6: /USB1+ -> Net-(J2-D+-PadA6)
- J2 pad B7: /USB1- -> Net-(J2-D--PadA7)
- J2 pad B9: VUSB -> Net-(U1-VBUS)
- J3 pad 1: VUSB -> /UART_TXD
- J3 pad 2: /Voltage Regulator/VIN -> /UART_RXD
- J3 pad 3: VIN -> GND
- J4 pad 1: Net-(J4-Pin_1) -> /CTL_SW1
- J4 pad 2: Net-(J4-Pin_2) -> /CTL_SW2
- L1 pad 1: Net-(U3-SW) -> Net-(U6-SW)
- R10 pad 1: /USB1+ -> +3.3V
- R10 pad 2: /USB+ -> Net-(U4-GPIO8)
- R11 pad 2: Net-(U1-GPIO9) -> Net-(U4-GPIO9)
- R2 pad 1: +5V -> Net-(J2-CC2)
- R2 pad 2: Net-(U3-FB) -> GND
- R3 pad 1: Net-(U3-FB) -> Net-(Q1-G)
- R3 pad 2: GND -> Net-(D2-A)
- R4 pad 1: Net-(U3-RT) -> Net-(D2-A)
- R5 pad 1: Net-(J5-CC2) -> Net-(R5-Pad1)
- R5 pad 2: GND -> /USB-
- R6 pad 1: +3.3V -> Net-(R6-Pad1)
- R6 pad 2: Net-(U1-EN/CHIP_PU) -> /USB+
- R7 pad 1: +3.3V -> /SWON
- R7 pad 2: Net-(U1-GPIO2/ADC1_CH2) -> Net-(R7-Pad2)
- R8 pad 2: Net-(U1-GPIO8) -> Net-(U4-EN/CHIP_PU)
- R9 pad 1: /USB1- -> +3.3V
- R9 pad 2: /USB- -> Net-(U4-GPIO2/ADC1_CH2)
- SW1 pad 2: Net-(U1-GPIO9) -> Net-(U4-EN/CHIP_PU)
- SW2 pad 2: Net-(U1-EN/CHIP_PU) -> Net-(U4-GPIO9)
- U2 pad 1: /RDR_TX -> Net-(R7-Pad2)
- U2 pad 2: /RDR_RX -> GND
- U2 pad 3: /OUT -> /CTL_SW2
- U2 pad 4: GND -> /CTL_SW1
- U3 pad 1: Net-(U3-BST) -> /RDR_TX
- U3 pad 2: Net-(U3-SW) -> /RDR_RX
- U3 pad 3: Net-(JP1-B) -> /OUT
- U3 pad 4: Net-(U3-RT) -> GND
- U3 pad 5: Net-(JP1-C) -> +5V
- U4 pad 16: unconnected-(U1-GPIO10-Pad16) -> /LED
- U4 pad 18: unconnected-(U1-GPIO4/ADC1_CH4-Pad18) -> /SWON
- U4 pad 22: Net-(U1-GPIO8) -> Net-(U4-GPIO8)
- U4 pad 23: Net-(U1-GPIO9) -> Net-(U4-GPIO9)
- U4 pad 30: Net-(J4-Pin_2) -> /UART_RXD
- U4 pad 31: Net-(J4-Pin_1) -> /UART_TXD
- U4 pad 5: Net-(U1-GPIO2/ADC1_CH2) -> Net-(U4-GPIO2/ADC1_CH2)
- U4 pad 6: unconnected-(U1-GPIO3/ADC1_CH3-Pad6) -> /STAT_SW
- U4 pad 8: Net-(U1-EN/CHIP_PU) -> Net-(U4-EN/CHIP_PU)
Routing:
- net +3.3V: track 0.00 -> 103.3 mm, vias 0 -> 2
- net /SWON: track 0.00 -> 83.8 mm, vias 0 -> 2
- net +5V: track 0.00 -> 81.3 mm, vias 0 -> 3
- net /OUT: track 0.00 -> 65.4 mm, vias 0 -> 1
- net /RDR_RX: track 0.00 -> 62.6 mm, vias 0 -> 2
- net /STAT_SW: track 0.00 -> 62.3 mm, vias 0 -> 1
- net /RDR_TX: track 0.00 -> 57.7 mm, vias 0 -> 2
- net Net-(U4-GPIO9): track 0.00 -> 48.3 mm, vias 0 -> 3
- net Net-(U4-EN/CHIP_PU): track 0.00 -> 41.4 mm, vias 0 -> 2
- net VIN: track 0.00 -> 33.1 mm
- net /UART_RXD: track 0.00 -> 28.0 mm
- net /UART_TXD: track 0.00 -> 24.3 mm
- net /LED: track 0.00 -> 23.7 mm, vias 0 -> 2
- net Net-(U4-GPIO8): track 0.00 -> 18.9 mm, vias 0 -> 2
- net Net-(U1-VBUS): track 0.00 -> 17.2 mm
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- added copper zone on B.Cu, net GND
- added copper zone on F.Cu, net GND
Other:
- board text added: "BOOT"
- board text added: "RST"

Commit message: Rev B Submitted
Parts:
- D1: value P6SMB24CA-E3/52 -> SMBJ16CA
- moved D1 0.14 mm to (86.4, 106.0)
Routing:
- net Net-(U4-EN/CHIP_PU): track 41.4 -> 42.3 mm
- net Net-(D4-DIN): track 14.7 -> 15.5 mm
- net /RDR_TX: track 57.7 -> 58.3 mm
- net GND: vias 332 -> 334
